File: EAGLE_files/electrosteel_2020/electrosteel2021_synthboards1.brd (EAGLE design)
At the start: 431.8 x 99.1 mm, 143 parts, among them IC1 OPA4344E, J1 4P-2.0, J2 4P-2.0, J3 4P-2.0, J36 4P-2.0, J4 4P-2.0, U1 MAX11615EEE+, U15 R-78E5.0-1.0, U17 R-78E5.0-1.0, U2 R-78E5.0-1.0, U20 TCA9548APWR, X6 2520-, X7 2516-

Commit message: working electrosteel, doesnt take in new patches but reads electrobass patches off sdcard
Connections:
- net N$298 renamed PA0-0
- net N$300 renamed PA2-0
Changed lines of the file:
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@@
 <wire x1="57.912" y1="54.864" x2="62.396" y2="54.864" width="0.254" layer="1"/>
 </signal>
-<signal name="N$298">
+<signal name="PA0-0">
 <contactref element="JP9" pad="13"/>
 <contactref element="JP1" pad="4"/>
@@
 <wire x1="125.73" y1="52.5526" x2="123.1646" y2="49.9872" width="0.254" layer="1"/>
 </signal>
-<signal name="N$300">
+<signal name="PA2-0">
 <contactref element="JP9" pad="15"/>
 <contactref element="JP1" pad="2"/>
