File: kicad_files/new_fretboard_rev1/_autosave-new_fretboard_rev1.kicad_pcb (KiCad board)
At the start: 2 copper layers, 635 x 114 mm, 22 parts, among them U2 LX3302AQPW-TR-EASY

Commit message: good single channel of fretboard rev
Routing:
- net GND: track 18.1 -> 21.2 mm, vias 9 -> 10
- net /CL2_A: track 11.0 -> 11.4 mm, vias 0 -> 2
