File: kicad_files/new_fretboard_rev1/new_fretboard_rev1.kicad_sch (KiCad schematic)
At the start: 28 parts, among them CN1 Header 1x6, J1 JMP, J2 JMP, J3 JMP, J4 JMP, U1 LX3302AQPW_TSSOP-14

Commit message: working on sensor circuit
Parts:
- removed C1, C10, C2, C7, C9: Capacitor NP, CAP_C_0603, symbol MCHP-CDB:root_2_Capacitor NP_MCHP-CDB.DbLib_0
- removed C11, C3, C4, C5, C6, C8: Capacitor NP, CAP_C_0603, symbol MCHP-CDB:root_1_Capacitor NP_MCHP-CDB.DbLib_0
- removed CN1: Header 1x6, HDR_M_2.54_1x6, symbol MCHP-CDB:root_3_Header 1x6_MCHP-CDB.DbLib_0
- removed J1, J2: JMP, JMP, symbol LX3301EVB1R1X1:root_0_JMP_LX3301EVB1R1X1.SCHLIB
- removed J3, J4: JMP, JMP, symbol LX3301EVB1R1X1:root_1_JMP_LX3301EVB1R1X1.SCHLIB
- removed L1, L2: PCB L, JMP, symbol Miscellaneous Devices:root_1_Inductor_Miscellaneous Devices.IntLib
- removed L3, L4: PCB L, JMP, symbol Miscellaneous Devices:root_0_Inductor_Miscellaneous Devices.IntLib
- removed R1, R5, R6, R7: Resistor, RES_C_0603, symbol MCHP-CDB:root_0_Resistor_MCHP-CDB.DbLib
- removed R2, R3, R4: Resistor, RES_C_0603, symbol MCHP-CDB:root_1_Resistor_MCHP-CDB.DbLib
- removed U1: LX3302AQPW_TSSOP-14, TSSOP-14, symbol MCHP-CDB:root_0_LX3302AQPW_TSSOP-14_MCHP-CDB.DbLib
- added C12, C13: 680pf, Capacitor_SMD:C_0603_1608Metric, symbol Device:C
- added C14, C15: 10pf, Capacitor_SMD:C_0402_1005Metric, symbol Device:C
- added C16: 1uf, Capacitor_SMD:C_0603_1608Metric, symbol Device:C
- added C17, C20: 100nf, Capacitor_SMD:C_0402_1005Metric, symbol Device:C
- added C18, C19: 6.8nf, Capacitor_SMD:C_0402_1005Metric, symbol Device:C
- added C21: 1000pf, Capacitor_SMD:C_0402_1005Metric, symbol Device:C
- added C22: 470nf, Capacitor_SMD:C_0402_1005Metric, symbol Device:C
- added L5, L6: L, symbol Device:L
- added L7, L8: L, Jumper:SolderJumper-2_P1.3mm_Bridged2Bar_RoundedPad1.0x1.5mm, symbol Device:L
- added R10, R11, R8, R9: 10R, Resistor_SMD:R_0402_1005Metric, symbol Device:R
- added R12: 221R, Resistor_SMD:R_0402_1005Metric, symbol Device:R
- added R13: 4.7R, Resistor_SMD:R_0402_1005Metric, symbol Device:R
- added U2: LX3302AQPW-TR-EASY, Snapeda:14-TSSOP_MCH-L, symbol Snapeda:LX3302AQPW-TR-EASY
Connections:
- new net: C16.2, C17.2, U2.5 (VDD)
- new net: C19.2, R11.1, R12.1, U2.6 (IO2)
- new net: C20.2, R13.2
- new net: C18.2, R12.2
- new net CL1B_A: L8.1, R10.2
- new net CL1_A: C15.1, R10.1, U2.8 (CL1)
- new net CL2B_A: L7.1, R9.2
- new net CL2_A: C14.1, R9.1, U2.10 (CL2)
- new net GND: C12.2, C13.2, C14.2, C15.2, C16.1, C18.1, C19.1, C20.1, C21.1, C22.1, L7.2, L8.2, U2.2 (GND), U2.9 (GNDCL)
- new net OSC11_A: C13.1, L5.2, U2.13 (OSC1)
- new net OSC12_A: C12.1, L6.2, U2.12 (OSC2)
- new net OSC2B_A: L5.1, L6.1, R8.2
- new net SUB_A: C17.1, U2.11 (SUB)
- new net VIN_A: C21.2, C22.2, R11.2, R13.1, R8.1, U2.4 (VIN)
Other:
- note removed: "${#} of ${##}"
- note removed: "${CURRENT_DATE}"
- note removed: "${FILENAME}"
- note removed: "${PROJECTDRAWNBY}"
- note removed: "${PROJECTENGINEER}"
- note removed: "${PROJECTPARTNUMBER}"
- note removed: "${PROJECTREVISIONART}"
- note removed: "${PROJECTREVISIONSCH}"
- note removed: "${PROJECTTITLE}"
- note removed: "${SHEETTITLE}"
- note removed: "${VARIANTNAME}"
- note removed: "03-${PROJECTPCBASSYNUMBER}"
- note removed: "04-${PROJECTPCBNUMBER}"
- note removed: "AOUT"
- note removed: "B"
- note removed: "Date:"
- note removed: "Designed with"
- note removed: "File:"
- note removed: "GND"
- note removed: "IOIN"
- note removed: "PCB #:"
- note removed: "PCB Layout Contact:"
- note removed: "PWMOUT"
- note removed: "PartNumber:"
- note removed: "Project Owner:"
- note removed: "Project Title"
- note removed: "Rev:"
- note removed: "SCH #:"
- note removed: "SENTOUT"
- note removed: "Sheet"
- note removed: "Sheet Title"
- note removed: "Size"
- note removed: "VIN"
- note removed: "Variant:"

Commit message: good single channel of fretboard rev
Parts:
- L5, L6: footprint (none) -> NetTie:NetTie-2_SMD_Pad0.5mm
- L7, L8: footprint Jumper:SolderJumper-2_P1.3mm_Bridged2Bar_RoundedPad1.0x1.5mm -> NetTie:NetTie-2_SMD_Pad0.5mm
Changed lines of the file:
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@@
 			)
 		)
-		(property "Footprint" ""
+		(property "Footprint" "NetTie:NetTie-2_SMD_Pad0.5mm"
 			(at 335.28 64.77 0)
 			(effects
@@
 			)
 		)
-		(property "Footprint" "Jumper:SolderJumper-2_P1.3mm_Bridged2Bar_RoundedPad1.0x1.5mm"
+		(property "Footprint" "NetTie:NetTie-2_SMD_Pad0.5mm"
 			(at 344.17 109.22 0)
 			(effects
@@
 			)
 		)
-		(property "Footprint" ""
+		(property "Footprint" "NetTie:NetTie-2_SMD_Pad0.5mm"
 			(at 325.12 64.77 0)
 			(effects
@@
 			)
 		)
-		(property "Footprint" "Jumper:SolderJumper-2_P1.3mm_Bridged2Bar_RoundedPad1.0x1.5mm"
+		(property "Footprint" "NetTie:NetTie-2_SMD_Pad0.5mm"
 			(at 344.17 118.11 0)
 			(effects
