File: kicad_files/new_fretboard_rev1/singlechannel_rev2.kicad_sch (KiCad schematic)
At the start: 22 parts, among them U2 LX3302AQPW-TR-EASY

Commit message: version with three coil circuits, some errors
Parts:
- removed C12, C13: 680pf, Capacitor_SMD:C_0603_1608Metric, symbol Device:C
- removed C14, C15: 10pf, Capacitor_SMD:C_0402_1005Metric, symbol Device:C
- removed C16: 1uf, Capacitor_SMD:C_0603_1608Metric, symbol Device:C
- removed C17, C20: 100nf, Capacitor_SMD:C_0402_1005Metric, symbol Device:C
- removed C18, C19: 6.8nf, Capacitor_SMD:C_0402_1005Metric, symbol Device:C
- removed C21: 1000pf, Capacitor_SMD:C_0402_1005Metric, symbol Device:C
- removed C22: 470nf, Capacitor_SMD:C_0402_1005Metric, symbol Device:C
- removed L5, L6, L7, L8: L, NetTie:NetTie-2_SMD_Pad0.5mm, symbol Device:L
- removed R10, R11, R8, R9: 10R, Resistor_SMD:R_0402_1005Metric, symbol Device:R
- removed R12: 221R, Resistor_SMD:R_0402_1005Metric, symbol Device:R
- removed R13: 4.7R, Resistor_SMD:R_0402_1005Metric, symbol Device:R
- removed U2: LX3302AQPW-TR-EASY, Snapeda:14-TSSOP_MCH-L, symbol Snapeda:LX3302AQPW-TR-EASY
- added C34, C40: 100nf, Capacitor_SMD:C_0402_1005Metric, symbol Device:C
- added C35: 1000pf, Capacitor_SMD:C_0402_1005Metric, symbol Device:C
- added C36: 470nf, Capacitor_SMD:C_0402_1005Metric, symbol Device:C
- added C37: 1uf, Capacitor_SMD:C_0603_1608Metric, symbol Device:C
- added C38, C39: 6.8nf, Capacitor_SMD:C_0402_1005Metric, symbol Device:C
- added C41, C42: 10pf, Capacitor_SMD:C_0402_1005Metric, symbol Device:C
- added C43, C44: 680pf, Capacitor_SMD:C_0603_1608Metric, symbol Device:C
- added L13, L14, L15, L16: L, NetTie:NetTie-2_SMD_Pad0.5mm, symbol Device:L
- added R19: 4.7R, Resistor_SMD:R_0402_1005Metric, symbol Device:R
- added R20: 221R, Resistor_SMD:R_0402_1005Metric, symbol Device:R
- added R21, R22, R23, R24: 10R, Resistor_SMD:R_0402_1005Metric, symbol Device:R
- added U4: LX3302AQPW-TR-EASY, Snapeda:14-TSSOP_MCH-L, symbol Snapeda:LX3302AQPW-TR-EASY
Connections:
- net CL1B_A: now also L16.1, R24.2
- net CL1_A: now also C41.1, R24.1, U4.8 (CL1)
- net CL2B_A: now also L15.1, R23.2
- net CL2_A: now also C42.1, R23.1, U4.10 (CL2)
- net GND: now also C34.1, C35.1, C36.1, C37.1, C38.1, C39.1, C41.2, C42.2, C43.2, C44.2, L15.2, L16.2, U4.2 (GND), U4.9 (GNDCL)
- net OSC11_A: now also C43.1, L13.2, U4.13 (OSC1)
- net OSC12_A: now also C44.1, L14.2, U4.12 (OSC2)
- net OSC2B_A: now also L13.1, L14.1, R22.2
- net SUB_A: now also C40.1, U4.11 (SUB)
- net VIN_A: now also C35.2, C36.2, R19.1, R21.2, R22.1, U4.4 (VIN)
- new net: C37.2, C40.2, U4.5 (VDD)
- new net: C38.2, R20.2
- new net: C39.2, R20.1, R21.1, U4.6 (IO2)
- new net: C34.2, R19.2
Other:
- removed sheet testchannel1
- removed sheet testchannel2
