File: kicad_files/new_fretboard_rev1/_autosave-new_fretboard_rev1.kicad_sch (KiCad schematic)
At the start: 22 parts, among them U2 LX3302AQPW-TR-EASY

Commit message: all circuit traces
Other:
- added sheet testchannel8 (testchannel8.kicad_sch)
Changed lines of the file:
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@@
+	)
+	(sheet
+		(at 508 182.88)
+		(size 82.55 62.23)
+		(exclude_from_sim no)
+		(in_bom yes)
+		(on_board yes)
+		(dnp no)
+		(fields_autoplaced yes)
+		(stroke
+			(width 0.1524)
+			(type solid)
+		)
+		(fill
+			(color 0 0 0 0.0000)
+		)
+		(property "Sheetname" "testchannel8"
+			(at 508 182.1684 0)
+			(effects
+				(font
+					(size 1.27 1.27)
+				)
+				(justify left bottom)
+			)
+		)
+		(property "Sheetfile" "testchannel8.kicad_sch"
+			(at 508 245.6946 0)
+			(effects
+				(font
+					(size 1.27 1.27)
+				)
+				(justify left top)
+			)
+		)
+		(instances
+			(project "new_fretboard_rev1"
+				(path "/bd5070b5-189c-4dfb-a5e7-79e743be8aa7"
+					(page "9")
+				)
+			)
+		)
 	)
 	(sheet
