File: kicad_files/new_fretboard_rev1/_autosave-testchannel8.kicad_sch (KiCad schematic)
At the start: 22 parts, among them U2 LX3302AQPW-TR-EASY

Commit message: all circuit traces
Parts:
- removed C12, C13: 680pf, Capacitor_SMD:C_0603_1608Metric, symbol Device:C
- removed C14, C15: 10pf, Capacitor_SMD:C_0402_1005Metric, symbol Device:C
- removed C16: 1uf, Capacitor_SMD:C_0603_1608Metric, symbol Device:C
- removed C17, C20: 100nf, Capacitor_SMD:C_0402_1005Metric, symbol Device:C
- removed C18, C19: 6.8nf, Capacitor_SMD:C_0402_1005Metric, symbol Device:C
- removed C21: 1000pf, Capacitor_SMD:C_0402_1005Metric, symbol Device:C
- removed C22: 470nf, Capacitor_SMD:C_0402_1005Metric, symbol Device:C
- removed L5, L6, L7, L8: L, NetTie:NetTie-2_SMD_Pad0.5mm, symbol Device:L
- removed R10, R11, R8, R9: 10R, Resistor_SMD:R_0402_1005Metric, symbol Device:R
- removed R12: 221R, Resistor_SMD:R_0402_1005Metric, symbol Device:R
- removed R13: 4.7R, Resistor_SMD:R_0402_1005Metric, symbol Device:R
- removed U2: LX3302AQPW-TR-EASY, Snapeda:14-TSSOP_MCH-L, symbol Snapeda:LX3302AQPW-TR-EASY
- added C89, C95: 100nf, Capacitor_SMD:C_0402_1005Metric, symbol Device:C
- added C90: 1000pf, Capacitor_SMD:C_0402_1005Metric, symbol Device:C
- added C91: 470nf, Capacitor_SMD:C_0402_1005Metric, symbol Device:C
- added C92: 1uf, Capacitor_SMD:C_0603_1608Metric, symbol Device:C
- added C93, C94: 6.8nf, Capacitor_SMD:C_0402_1005Metric, symbol Device:C
- added C96, C97: 10pf, Capacitor_SMD:C_0402_1005Metric, symbol Device:C
- added C98, C99: 680pf, Capacitor_SMD:C_0603_1608Metric, symbol Device:C
- added L33, L34, L35, L36: L, NetTie:NetTie-2_SMD_Pad0.5mm, symbol Device:L
- added R49: 4.7R, Resistor_SMD:R_0402_1005Metric, symbol Device:R
- added R50: 221R, Resistor_SMD:R_0402_1005Metric, symbol Device:R
- added R51, R52, R53, R54: 10R, Resistor_SMD:R_0402_1005Metric, symbol Device:R
- added U9: LX3302AQPW-TR-EASY, Snapeda:14-TSSOP_MCH-L, symbol Snapeda:LX3302AQPW-TR-EASY
Connections:
- net CL1B_A: now also L36.1, R54.2
- net CL1_A: now also C96.1, R54.1, U9.8 (CL1)
- net CL2B_A: now also L35.1, R53.2
- net CL2_A: now also C97.1, R53.1, U9.10 (CL2)
- net GND: now also C89.1, C90.1, C91.1, C92.1, C93.1, C94.1, C96.2, C97.2, C98.2, C99.2, L35.2, L36.2, U9.2 (GND), U9.9 (GNDCL)
- net OSC11_A: now also C98.1, L33.2, U9.13 (OSC1)
- net OSC12_A: now also C99.1, L34.2, U9.12 (OSC2)
- net SUB_A: now also C95.1, U9.11 (SUB)
- net VIN_A: now also C90.2, C91.2, R49.1, R51.2, R52.1, U9.4 (VIN)
- new net: C92.2, C95.2, U9.5 (VDD)
- new net: C94.2, R50.1, R51.1, U9.6 (IO2)
- new net: C93.2, R50.2
- new net: C89.2, R49.2
- new net /OSC2B_A: L33.1, L34.1, R52.2
Other:
- removed sheet testchannel1
- removed sheet testchannel2
- removed sheet testchannel3
- removed sheet testchannel4
- removed sheet testchannel5
- removed sheet testchannel6
- removed sheet testchannel7
