File: kicad_files/new_fretboard_rev1/new_fretboard_rev1.kicad_pcb (KiCad board)
At the start: 2 copper layers, 635 x 114 mm, 198 parts, among them U1 LX3302AQPW-TR-EASY, U2 LX3302AQPW-TR-EASY, U3 LX3302AQPW-TR-EASY, U4 LX3302AQPW-TR-EASY, U5 LX3302AQPW-TR-EASY, U6 LX3302AQPW-TR-EASY, U7 LX3302AQPW-TR-EASY, U8 LX3302AQPW-TR-EASY, U9 LX3302AQPW-TR-EASY

Commit message: all circuit traces, fixed circuit 2
Parts:
- moved C10 141.7 mm to (64.6, 188.4)
- moved C11 141.7 mm to (64.6, 189.9)
- moved C4 141.7 mm to (64.8, 193.4)
- moved C5 141.7 mm to (61.8, 191.6)
- moved C6 141.7 mm to (62.6, 193.1)
- moved C7 141.7 mm to (65.6, 191.6)
- moved L1 141.7 mm to (80.3, 190.7)
- moved R2 141.7 mm to (61.3, 193.1)
- moved R3 141.7 mm to (73.3, 192.6)
- moved R4 141.7 mm to (73.3, 191.4)
- moved R5 141.7 mm to (73.3, 190.1)
- moved U1 141.7 mm to (69.3, 190.6)
- moved C1 141.7 mm to (59.9, 193.2)
- moved C2 141.7 mm to (59.9, 189.7)
- moved C3 141.7 mm to (61.2, 189.7)
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Routing:
- net /testchannel1/OSC11_A: track 2124.7 -> 2112.1 mm, vias 6 -> 4
- net /testchannel1//OSC2B_A: track 0.00 -> 12.6 mm, vias 0 -> 2
