File: kicad_files/new_fretboard_rev1/new_fretboard_rev1.kicad_pcb (KiCad board)
At the start: 2 copper layers, 635 x 114 mm, 303 parts, among them J1 530470410, J10 530470410, J11 110990030, J12 110990030, J13 110990030, J2 530470410, J3 FTSH-107-01-L-DV-K-A, J4 530470410, J5 530470410, J6 530470410, J7 530470410, J8 530470410, J9 530470410, U1 LX3302AQPW-TR-EASY, U10 STM32F730V8Tx, U11 MIC5504-3.3YM5, U2 LX3302AQPW-TR-EASY, U3 LX3302AQPW-TR-EASY, U4 LX3302AQPW-TR-EASY, U5 LX3302AQPW-TR-EASY, U6 LX3302AQPW-TR-EASY, U7 LX3302AQPW-TR-EASY, U8 LX3302AQPW-TR-EASY, U9 LX3302AQPW-TR-EASY, Y1 ASE-25.000MHZ-LC-T

Commit message: mostly done, adjusting silkscreen labels
Parts:
- removed H14, H15, H16, H17, H18, H19, H20: MountingHole, MountingHole:MountingHole_2.1mm
- moved H12 64.8 mm to (572.5, 139.5)
- moved H13 22.7 mm to (572.6, 105.2)
- moved H11 9.08 mm to (572.5, 71.0)
- turned L13 to -89.86 degrees
- turned L14 to 0.14 degrees
- turned H5 to -0.01 degrees
- turned H4 to -0.01 degrees
Other:
- board size 635 x 114 mm -> 576.1 x 81.9 mm
