File: kicad_files/new_fretboard_rev1/_autosave-testchannel1.kicad_sch (KiCad schematic)
At the start: 22 parts, among them U2 LX3302AQPW-TR-EASY

Commit message: all circuit traces,in position
Parts:
- removed C12, C13: 680pf, Capacitor_SMD:C_0603_1608Metric, symbol Device:C
- removed C14, C15: 10pf, Capacitor_SMD:C_0402_1005Metric, symbol Device:C
- removed C16: 1uf, Capacitor_SMD:C_0603_1608Metric, symbol Device:C
- removed C17, C20: 100nf, Capacitor_SMD:C_0402_1005Metric, symbol Device:C
- removed C18, C19: 6.8nf, Capacitor_SMD:C_0402_1005Metric, symbol Device:C
- removed C21: 1000pf, Capacitor_SMD:C_0402_1005Metric, symbol Device:C
- removed C22: 470nf, Capacitor_SMD:C_0402_1005Metric, symbol Device:C
- removed L5, L6, L7, L8: L, NetTie:NetTie-2_SMD_Pad0.5mm, symbol Device:L
- removed R10, R11, R8, R9: 10R, Resistor_SMD:R_0402_1005Metric, symbol Device:R
- removed R12: 221R, Resistor_SMD:R_0402_1005Metric, symbol Device:R
- removed R13: 4.7R, Resistor_SMD:R_0402_1005Metric, symbol Device:R
- removed U2: LX3302AQPW-TR-EASY, Snapeda:14-TSSOP_MCH-L, symbol Snapeda:LX3302AQPW-TR-EASY
- added C1, C7: 100nf, Capacitor_SMD:C_0402_1005Metric, symbol Device:C
- added C10, C11: 680pf, Capacitor_SMD:C_0603_1608Metric, symbol Device:C
- added C2: 1000pf, Capacitor_SMD:C_0402_1005Metric, symbol Device:C
- added C3: 470nf, Capacitor_SMD:C_0402_1005Metric, symbol Device:C
- added C4: 1uf, Capacitor_SMD:C_0603_1608Metric, symbol Device:C
- added C5, C6: 6.8nf, Capacitor_SMD:C_0402_1005Metric, symbol Device:C
- added C8, C9: 10pf, Capacitor_SMD:C_0402_1005Metric, symbol Device:C
- added L1, L2, L3, L4: L, NetTie:NetTie-2_SMD_Pad0.5mm, symbol Device:L
- added R1: 4.7R, Resistor_SMD:R_0402_1005Metric, symbol Device:R
- added R2: 221R, Resistor_SMD:R_0402_1005Metric, symbol Device:R
- added R3, R4, R5, R6: 10R, Resistor_SMD:R_0402_1005Metric, symbol Device:R
- added U1: LX3302AQPW-TR-EASY, Snapeda:14-TSSOP_MCH-L, symbol Snapeda:LX3302AQPW-TR-EASY
Connections:
- net CL1B_A: now also L4.1, R6.2
- net CL1_A: now also C8.1, R6.1, U1.8 (CL1)
- net CL2B_A: now also L3.1, R5.2
- net CL2_A: now also C9.1, R5.1, U1.10 (CL2)
- net GND: now also C1.1, C10.2, C11.2, C2.1, C3.1, C4.1, C5.1, C6.1, C8.2, C9.2, L3.2, L4.2, U1.2 (GND), U1.9 (GNDCL)
- net OSC11_A: now also C10.1, L1.2, U1.13 (OSC1)
- net OSC12_A: now also C11.1, L2.2, U1.12 (OSC2)
- net SUB_A: now also C7.1, U1.11 (SUB)
- net VIN_A: now also C2.2, C3.2, R1.1, R3.2, R4.1, U1.4 (VIN)
- new net: C4.2, C7.2, U1.5 (VDD)
- new net: C6.2, R2.1, R3.1, U1.6 (IO2)
- new net: C5.2, R2.2
- new net: C1.2, R1.2
- new net /OSC2B_A: L1.1, L2.1, R4.2
Other:
- removed sheet testchannel1
- removed sheet testchannel2
- removed sheet testchannel3
- removed sheet testchannel4
- removed sheet testchannel5
- removed sheet testchannel6
- removed sheet testchannel7
- removed sheet testchannel8
