File: kicad_files/new_fretboard_rev1/_autosave-testchannel2.kicad_sch (KiCad schematic)
At the start: 22 parts, among them U2 LX3302AQPW-TR-EASY

Commit message: all circuit traces,in position
Parts:
- removed C12, C13: 680pf, Capacitor_SMD:C_0603_1608Metric, symbol Device:C
- removed C14, C15: 10pf, Capacitor_SMD:C_0402_1005Metric, symbol Device:C
- removed C16: 1uf, Capacitor_SMD:C_0603_1608Metric, symbol Device:C
- removed C17, C20: 100nf, Capacitor_SMD:C_0402_1005Metric, symbol Device:C
- removed C18, C19: 6.8nf, Capacitor_SMD:C_0402_1005Metric, symbol Device:C
- removed C21: 1000pf, Capacitor_SMD:C_0402_1005Metric, symbol Device:C
- removed C22: 470nf, Capacitor_SMD:C_0402_1005Metric, symbol Device:C
- removed L5, L6, L7, L8: L, NetTie:NetTie-2_SMD_Pad0.5mm, symbol Device:L
- removed R10, R11, R8, R9: 10R, Resistor_SMD:R_0402_1005Metric, symbol Device:R
- removed R12: 221R, Resistor_SMD:R_0402_1005Metric, symbol Device:R
- removed R13: 4.7R, Resistor_SMD:R_0402_1005Metric, symbol Device:R
- removed U2: LX3302AQPW-TR-EASY, Snapeda:14-TSSOP_MCH-L, symbol Snapeda:LX3302AQPW-TR-EASY
- added C23, C29: 100nf, Capacitor_SMD:C_0402_1005Metric, symbol Device:C
- added C24: 1000pf, Capacitor_SMD:C_0402_1005Metric, symbol Device:C
- added C25: 470nf, Capacitor_SMD:C_0402_1005Metric, symbol Device:C
- added C26: 1uf, Capacitor_SMD:C_0603_1608Metric, symbol Device:C
- added C27, C28: 6.8nf, Capacitor_SMD:C_0402_1005Metric, symbol Device:C
- added C30, C31: 10pf, Capacitor_SMD:C_0402_1005Metric, symbol Device:C
- added C32, C33: 680pf, Capacitor_SMD:C_0603_1608Metric, symbol Device:C
- added L10, L11, L12, L9: L, NetTie:NetTie-2_SMD_Pad0.5mm, symbol Device:L
- added R14: 221R, Resistor_SMD:R_0402_1005Metric, symbol Device:R
- added R15, R16, R17, R18: 10R, Resistor_SMD:R_0402_1005Metric, symbol Device:R
- added R7: 4.7R, Resistor_SMD:R_0402_1005Metric, symbol Device:R
- added U3: LX3302AQPW-TR-EASY, Snapeda:14-TSSOP_MCH-L, symbol Snapeda:LX3302AQPW-TR-EASY
Connections:
- net CL1B_A: now also L12.1, R18.2
- net CL1_A: now also C30.1, R18.1, U3.8 (CL1)
- net CL2B_A: now also L11.1, R17.2
- net CL2_A: now also C31.1, R17.1, U3.10 (CL2)
- net GND: now also C23.1, C24.1, C25.1, C26.1, C27.1, C28.1, C30.2, C31.2, C32.2, C33.2, L11.2, L12.2, U3.2 (GND), U3.9 (GNDCL)
- net OSC11_A: now also C32.1, L9.2, U3.13 (OSC1)
- net OSC12_A: now also C33.1, L10.2, U3.12 (OSC2)
- net SUB_A: now also C29.1, U3.11 (SUB)
- net VIN_A: now also C24.2, C25.2, R15.2, R16.1, R7.1, U3.4 (VIN)
- new net: C26.2, C29.2, U3.5 (VDD)
- new net: C23.2, R7.2
- new net: C28.2, R14.1, R15.1, U3.6 (IO2)
- new net: C27.2, R14.2
- new net /OSC2B_A: L10.1, L9.1, R16.2
Other:
- removed sheet testchannel1
- removed sheet testchannel2
- removed sheet testchannel3
- removed sheet testchannel4
- removed sheet testchannel5
- removed sheet testchannel6
- removed sheet testchannel7
- removed sheet testchannel8
