File: kicad_files/new_fretboard_rev1/_autosave-testchannel5.kicad_sch (KiCad schematic)
At the start: 22 parts, among them U2 LX3302AQPW-TR-EASY

Commit message: all circuit traces,in position
Parts:
- removed C12, C13: 680pf, Capacitor_SMD:C_0603_1608Metric, symbol Device:C
- removed C14, C15: 10pf, Capacitor_SMD:C_0402_1005Metric, symbol Device:C
- removed C16: 1uf, Capacitor_SMD:C_0603_1608Metric, symbol Device:C
- removed C17, C20: 100nf, Capacitor_SMD:C_0402_1005Metric, symbol Device:C
- removed C18, C19: 6.8nf, Capacitor_SMD:C_0402_1005Metric, symbol Device:C
- removed C21: 1000pf, Capacitor_SMD:C_0402_1005Metric, symbol Device:C
- removed C22: 470nf, Capacitor_SMD:C_0402_1005Metric, symbol Device:C
- removed L5, L6, L7, L8: L, NetTie:NetTie-2_SMD_Pad0.5mm, symbol Device:L
- removed R10, R11, R8, R9: 10R, Resistor_SMD:R_0402_1005Metric, symbol Device:R
- removed R12: 221R, Resistor_SMD:R_0402_1005Metric, symbol Device:R
- removed R13: 4.7R, Resistor_SMD:R_0402_1005Metric, symbol Device:R
- removed U2: LX3302AQPW-TR-EASY, Snapeda:14-TSSOP_MCH-L, symbol Snapeda:LX3302AQPW-TR-EASY
- added C56, C62: 100nf, Capacitor_SMD:C_0402_1005Metric, symbol Device:C
- added C57: 1000pf, Capacitor_SMD:C_0402_1005Metric, symbol Device:C
- added C58: 470nf, Capacitor_SMD:C_0402_1005Metric, symbol Device:C
- added C59: 1uf, Capacitor_SMD:C_0603_1608Metric, symbol Device:C
- added C60, C61: 6.8nf, Capacitor_SMD:C_0402_1005Metric, symbol Device:C
- added C63, C64: 10pf, Capacitor_SMD:C_0402_1005Metric, symbol Device:C
- added C65, C66: 680pf, Capacitor_SMD:C_0603_1608Metric, symbol Device:C
- added L21, L22, L23, L24: L, NetTie:NetTie-2_SMD_Pad0.5mm, symbol Device:L
- added R31: 4.7R, Resistor_SMD:R_0402_1005Metric, symbol Device:R
- added R32: 221R, Resistor_SMD:R_0402_1005Metric, symbol Device:R
- added R33, R34, R35, R36: 10R, Resistor_SMD:R_0402_1005Metric, symbol Device:R
- added U6: LX3302AQPW-TR-EASY, Snapeda:14-TSSOP_MCH-L, symbol Snapeda:LX3302AQPW-TR-EASY
Connections:
- net CL1B_A: now also L24.1, R36.2
- net CL1_A: now also C63.1, R36.1, U6.8 (CL1)
- net CL2B_A: now also L23.1, R35.2
- net CL2_A: now also C64.1, R35.1, U6.10 (CL2)
- net GND: now also C56.1, C57.1, C58.1, C59.1, C60.1, C61.1, C63.2, C64.2, C65.2, C66.2, L23.2, L24.2, U6.2 (GND), U6.9 (GNDCL)
- net OSC11_A: now also C65.1, L21.2, U6.13 (OSC1)
- net OSC12_A: now also C66.1, L22.2, U6.12 (OSC2)
- net SUB_A: now also C62.1, U6.11 (SUB)
- net VIN_A: now also C57.2, C58.2, R31.1, R33.2, R34.1, U6.4 (VIN)
- new net: C60.2, R32.2
- new net: C61.2, R32.1, R33.1, U6.6 (IO2)
- new net: C56.2, R31.2
- new net: C59.2, C62.2, U6.5 (VDD)
- new net /OSC2B_A: L21.1, L22.1, R34.2
Other:
- removed sheet testchannel1
- removed sheet testchannel2
- removed sheet testchannel3
- removed sheet testchannel4
- removed sheet testchannel5
- removed sheet testchannel6
- removed sheet testchannel7
- removed sheet testchannel8
