File: kicad_files/electrosteel2020_10_arrange5.kicad_pcb (KiCad board)
At the start: 4 copper layers, 270.5 x 242.3 mm, 766 parts, among them IC1 OPA4344E, IC10 OPA4344E, IC11 LP5912, IC12 REG1117, IC13 REG1117, IC14 REG1117, IC15 REG1117, IC16 OPA4344E, IC17 OPA4344E, IC18 REG1117, IC2 LMV321M5, IC20 REG1117, IC3 STM32H743ZIT6, IC4 LMV321M5, IC7 OPA4344E, IC8 OPA4344E, IC9 OPA4344E, J1 AUDIO_JACK_TRS_0.25"_PTH_RA, J10 4P-2.0, J11 4P-2.0, J12 4P-2.0, J13 4P-2.0, J14 4P-2.0, J15 4P-2.0, J16 4P-2.0, J17 4P-2.0, J18 4P-2.0, J19 4P-2.0, J2 4P-2.0, J20 4P-2.0, J21 4P-2.0, J22 4P-2.0, J23 4P-2.0, J24 4P-2.0, J25 4P-2.0-90D, J26 4P-2.0, J27 4P-2.0-90D, J28 PJ-066A, J29 4P-2.0-90D, J3 4P-2.0, J31 4P-2.0-90D, J32 AUDIO_JACK_TRS_0.25"_PTH_RA, J33 4P-2.0-90D, J34 4P-2.0, J35 4P-2.0-90D, J36 4P-2.0, J37 4P-2.0-90D, J38 4P-2.0, J39 4P-2.0-90D, J4 4P-2.0, J41 4P-2.0-90D, J42 J-20-100-2X10_M, J5 4P-2.0, J6 4P-2.0, J7 4P-2.0, J8 4P-2.0, J9 4P-2.0-90D, P1 P-10-100-2X05_M, P2 P-24-100-2X12_M, P3 M-1X03-SIP-100-40Y, P4 M-1X03-SIP-100-40Y, Q1 25MHz, SW1 PEC11R-4215F-S0024, U1 CY8C5868AXI-LP035, U15 R-78E5.0-1.0, U16 TEXAS_TPS2051B, U17 R-78E5.0-1.0, U19 TCA9548APWR, U2 CY8C5868AXI-LP035, U20 TCA9548APWR, U22 AS5600, U23 AS5600, U25 AS5600, U27 AS5600, U29 AS5600, U31 AS5600, U33 AS5600, U35 AS5600, U37 AS5600, U39 AS5600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

Commit message: exported gerbers of lefthand
Parts:
- added R210: 1.5k, R0603_16378527, F.Cu at (146.6, 87.5)
- added R215: 1.5k, R0603_16378527, F.Cu at (138.7, 85.2)
- added SC7: , 1X01, F.Cu at (141.8, 83.7)
- added SD7: , 1X01, F.Cu at (141.8, 81.1)
Connections:
- U19 pad 19: (no net) -> N$311
- U19 pad 20: (no net) -> N$312
Routing:
- net N$311: track 0.00 -> 9.58 mm
- net N$312: track 0.00 -> 8.83 mm
- net 3V3D5: track 68.9 -> 73.7 mm, vias 13 -> 14
- net SDA_B: track 21.4 -> 22.4 mm
- net SCL_B: track 21.4 -> 22.2 mm
